Commit message: wip

File: ros2_ws/src/soarm_description/urdf/so101.urdf.xacro (robot description, xacro)
@@ -16,4 +16,12 @@
   <xacro:property name="mesh_path" value="package://soarm_description/meshes"/>
   <!-- ================================================================== -->
+  <!-- World fixation (screwed to the table)                              -->
+  <!-- ================================================================== -->
+  <link name="world"/>
+  <joint name="world_to_base" type="fixed">
+    <parent link="world"/>
+    <child link="base_link"/>
+  </joint>
+  <!-- ================================================================== -->
   <!-- Links                                                              -->
   <!-- ================================================================== -->
